File: control-pcb/control-pcb.sch (KiCad schematic (older format))
At the start: 7 parts, among them J0 Conn_01x15_Female, J1 Conn_01x15_Female, J2 Conn_01x04_Female

Commit message: Updated pcb
Parts:
- added J3, J4, J5: Conn_01x03_Female, Connector_PinHeader_2.54mm:PinHeader_1x03_P2.54mm_Vertical, symbol Connector:Conn_01x03_Female
- added R0, R1, R2, R3: 10k, Resistor_SMD:R_1206_3216Metric, symbol Device:R
- added SW0: SW_DIP_x01, Button_Switch_SMD:SW_DPDT_CK_JS202011JCQN, symbol Switch:SW_DIP_x01
- C0, C1: footprint (none) -> Capacitor_SMD:C_0603_1608Metric
- J0, J1: footprint (none) -> Connector_PinHeader_2.54mm:PinHeader_1x15_P2.54mm_Vertical
- J2: footprint (none) -> Connector_PinHeader_2.54mm:PinHeader_1x04_P2.54mm_Vertical
- J6: renamed from J?; footprint (none) -> Connector_BarrelJack:BarrelJack_Horizontal
- U0: renamed from U?; footprint (none) -> Connector_PinHeader_2.54mm:PinHeader_1x03_P2.54mm_Vertical
Connections:
- net +12V: now also J4.1 (Pin_1), J5.1 (Pin_1), SW0.2; no longer J6.1
- net +5V: now also J3.1 (Pin_1)
- net GND: now also J0.2 (Pin_2), J2.2 (Pin_2), J3.3 (Pin_3), J4.3 (Pin_3), J5.3 (Pin_3), R1.1, R3.1
- net at J1.11 (Pin_11): now also J3.2 (Pin_2)
- net at J1.12 (Pin_12): now also R0.2
- net at J1.13 (Pin_13): now also R2.2
- new net: J6.1, SW0.1
- new net: J4.2 (Pin_2), R0.1, R1.2
- new net: J5.2 (Pin_2), R2.1, R3.2
Other:
- moved on the sheet: C0, C1, J2, J6, U0
